Commit message: add basic example

File: src/config_files/reachy2.urdf (robot description, URDF)
Before this commit: robot reachy_v2, 44 links, 43 joints
Links:
- link r_gripper_palm_link: geometry collision box size=0.03 0.06 0.06; visual box size=0.03 0.06 0.06
Joints:
- joint r_gripper_finger: origin xyz=0 0.03 0.11 rpy=0 0 0 -> xyz=0 0.03 0.06 rpy=0 0 0
- joint r_gripper_finger_mimic: origin xyz=0 -0.03 0.11 rpy=0 0 0 -> xyz=0 -0.03 0.06 rpy=0 0 0
- joint r_shoulder_roll: limit lower=-2.6179938779914944 upper=0.6981317007977318 effort=1000.0 velocity=100.0 -> lower=-2.792526803190927 upper=0.0 effort=1000.0 velocity=100.0
- joint r_tip_joint: origin xyz=0 0 0.15 rpy=3.141592653589793 0 0 -> xyz=0 0 0.1 rpy=3.141592653589793 0 0
- joint r_wrist_roll: axis 1 0 0 -> 0 0 1; limit lower=-0.7853981633974483 upper=0.7853981633974483 effort=1000.0 velocity=100.0 -> lower=-6.283185307179586 upper=6.283185307179586 effort=1000.0 velocity=100.0

Commit message: add left arm

File: src/config_files/reachy2.urdf (robot description, URDF)
Before this commit: robot reachy_v2, 44 links, 43 joints
Joints:
- joint l_elbow_pitch: limit lower=-2.25 upper=0.1 effort=1000.0 velocity=100.0 -> lower=-2.2689280275926285 upper=0.0 effort=1000.0 velocity=100.0
- joint l_elbow_yaw: limit lower=-1.5707963267948966 upper=1.5707963267948966 effort=1000.0 velocity=100.0 -> lower=-6.283185307179586 upper=6.283185307179586 effort=1000.0 velocity=100.0
- joint l_shoulder_pitch: limit lower=-1.5707963267948966 upper=1.5707963267948966 effort=1000.0 velocity=100.0 -> lower=-6.283185307179586 upper=6.283185307179586 effort=1000.0 velocity=100.0; origin xyz=-0.0479 0.1913 0.025 rpy=0 0 -0.2617993877991494 -> xyz=0 0.2 0 rpy=-0.17453292519943295 0 -0.2617993877991494
- joint l_shoulder_roll: limit lower=-1.5707963267948966 upper=0.0 effort=1000.0 velocity=100.0 -> lower=0 upper=2.792526803190927 effort=1000.0 velocity=100.0
- joint l_wrist_pitch: limit lower=-0.35 upper=0.35 effort=1000.0 velocity=100.0 -> lower=-0.7853981633974483 upper=0.7853981633974483 effort=1000.0 velocity=100.0
- joint l_wrist_roll: axis 1 0 0 -> 0 0 1; limit lower=-0.35 upper=0.35 effort=1000.0 velocity=100.0 -> lower=-6.283185307179586 upper=6.283185307179586 effort=1000.0 velocity=100.0
- joint l_wrist_yaw: limit lower=-1.57 upper=1.57 effort=1000.0 velocity=100.0 -> lower=-6.283185307179586 upper=6.283185307179586 effort=1000.0 velocity=100.0

Commit message: add new tests

File: src/config_files/reachy2.urdf (robot description, URDF)
Before this commit: robot reachy2, 78 links, 77 joints
Joints:
- joint l_shoulder_base_joint: origin xyz=0.0 0.2 0.0 rpy=-1.7453292519943295 0 -0.2617993877991494 -> xyz=0.0 0.2 0.0 rpy=-1.3089969389957472 0 -0.17453292519943295
- joint r_shoulder_base_joint: origin xyz=0.0 -0.2 0.0 rpy=1.7453292519943295 0 0.2617993877991494 -> xyz=0.0 -0.2 0.0 rpy=1.3089969389957472 0 0.17453292519943295
